File: PCB/KeepCalm/KeepCalm.kicad_pcb (KiCad board)
At the start: 2 copper layers, 33 x 33 mm, 28 parts, among them SW1 SW_Push, U1 ATtiny85-20SU

Commit message: Final Changes To PCB
Parts:
- moved C1 0.51 mm to (159.0, 94.0)
- moved SW1 0.13 mm to (152.4, 82.5)
Routing:
- net +BATT: track 24.4 -> 27.3 mm
- net Net-(D1-Pad1): track 61.2 -> 62.0 mm
- net Net-(D11-Pad1): track 45.7 -> 46.3 mm
- net PIN0: track 22.9 -> 22.3 mm

Commit message: Basic Led Struct
Parts:
- moved U1 0.90 mm to (152.4, 95.5)
Routing:
- net PIN1: track 13.1 -> 15.5 mm
- net GND: track 49.3 -> 50.3 mm
- net PIN0: track 22.3 -> 23.3 mm
- net +BATT: track 27.3 -> 28.2 mm
